Commit message: Update urdf

File: xarm_urdf/urdf/xarm.urdf (robot description, URDF)
Before this commit: robot xarm, 13 links, 12 joints
Links:
- link base_link: geometry collision mesh filename=../meshes/base_link.glb; visual mesh filename=../meshes/base_link.glb
- link camera: geometry visual mesh filename=../meshes/camera_wrist.glb
- link camera_mount: geometry visual mesh filename=../meshes/camera_link.glb
- link gripper_base: geometry collision mesh filename=../meshes/gripper_base.glb; visual mesh filename=../meshes/gripper_base.glb
- link link1: geometry collision mesh filename=../meshes/link1.glb; visual mesh filename=../meshes/link1.glb
- link link2: geometry collision mesh filename=../meshes/link2.glb; visual mesh filename=../meshes/link2.dae
- link link3: geometry collision mesh filename=../meshes/link3.glb; visual mesh filename=../meshes/link3.glb
- link link4: geometry collision mesh filename=../meshes/link4.glb; visual mesh filename=../meshes/link4.glb
- link link5: geometry collision mesh filename=../meshes/link5.glb; visual mesh filename=../meshes/link5.glb
- link link6: geometry collision mesh filename=../meshes/link6.glb; visual mesh filename=../meshes/link6.glb
